Commit message: Add build log for April 18, 2025 and update latest build reference
- Created a new log file for the build executed on April 18, 2025.
- Updated the latest_build reference to point to the new log file.

Refactor ackermann_control.yaml configuration

- Removed redundant rear_wheels_radius entry and cleaned up comments in ackermann_control.yaml.

Comment out teleop_twist_keyboard node in rviz_launch.launch.py

- Temporarily disabled the teleop_twist_keyboard node to prevent it from launching during simulation.

Update base_link.xacro with joint configurations

- Added commented-out transmission configurations for motors and steering joints in base_link.xacro.
- Organized joint definitions for rear wheels and steering hinges for clarity.

Add keyboard_teleop as a subproject

- Introduced keyboard_teleop as a new subproject with the latest commit reference.

File: install/car_description/share/car_description/urdf/base_link.xacro (robot description, xacro)
@@ -1 +1,214 @@
-/home/ezo/f1tenth_ws/build/car_description/urdf/base_link.xacro
+<?xml version="1.0"?>
+<robot name="racecar" xmlns:xacro="http://www.ros.org/wiki/xacro">
+    <xacro:include filename="$(find car_description)/urdf/macros.xacro" />
+    <link name="base_link"/>
+<!-- Add the chassis with its joints -->
+    <link name="chassis">
+        <visual>
+            <xacro:chassis_geometry/>
+        </visual>
+        <collision>
+            <xacro:chassis_geometry/>
+        </collision>
+        <inertial>
+            <xacro:chassis_inertial_params />
+        </inertial>
+    </link>
+    <joint name="base_link_joint" type="fixed">
+        <origin xyz="0 0 0" rpy="0 0 0" />
+        <parent link="base_link" />
+        <child link="chassis" />
+    </joint>
+<!-- Add the rear wheels with their joints -->
+    <link name="left_rear_wheel">
+        <inertial>
+            <xacro:wheels_inertial_params z_offset="0" />
+        </inertial>
+        <visual>
+            <xacro:wheel_geometry prefix="left_rear" />
+        </visual>
+        <collision>
+            <xacro:wheel_collision_geometry />
+        </collision>
+    </link>
+    <joint name="left_rear_wheel_joint" type="continuous">
+        <origin xyz="${wheelbase/2} ${wheel_separation/2} 0.02" rpy="${pi/2} 0 0" />
+        <parent link="chassis" />
+        <child link="left_rear_wheel" />
+        <axis xyz="0 1 0" />
+        <limit effort="10" velocity="100" />
+    </joint>
+    <link name="right_rear_wheel">
+        <inertial>
+            <xacro:wheels_inertial_params z_offset="0" />
+        </inertial>
+        <visual>
+            <xacro:wheel_geometry prefix="right_rear" />
+        </visual>
+        <collision>
+            <xacro:wheel_collision_geometry />
+        </collision>
+    </link>
+    <joint name="right_rear_wheel_joint" type="continuous">
+        <origin xyz="${-wheelbase/2} ${wheel_separation/2} 0.02" rpy="${pi/2} 0 ${pi}" />
+        <parent link="chassis" />
+        <child link="right_rear_wheel" />
+        <axis xyz="0 1 0" />
+        <limit effort="10" velocity="100" />
+    </joint>
+    <link name="left_steering_hinge">
+        <inertial>
+            <xacro:steering_hinge_inertial_params z_offset="0"/>
+        </inertial>
+        <visual>
+            <xacro:steering_hinge_geometry prefix="left" />
+        </visual>
+         <collision>
+              <xacro:steering_hinge_geometry prefix="left" />
+        </collision>
+    </link>
+    <joint name="left_steering_hinge_joint" type="revolute">
+        <origin xyz="${wheelbase/2} ${-wheel_separation/2} 0.02" rpy="0 0 0" />
+        <parent link="chassis" />
+        <child link="left_steering_hinge" />
+        <axis xyz="0 0 1" />
+        <limit lower="-0.785" upper="0.785" effort="10" velocity="10" />
+    </joint>
+    <link name="right_steering_hinge">
+        <inertial>
+            <xacro:steering_hinge_inertial_params z_offset="0"/>
+        </inertial>
+        <visual>
+            <xacro:steering_hinge_geometry prefix="right" />
+        </visual>
+        <collision>
+            <xacro:steering_hinge_geometry prefix="right" />
+        </collision>
+    </link>
+    <joint name="right_steering_hinge_joint" type="revolute">
+        <origin xyz="${-wheelbase/2} ${-wheel_separation/2} 0.02" rpy="0 0 0" />
+        <parent link="chassis" />
+        <child link="right_steering_hinge" />
+        <axis xyz="0 0 1" />
+        <limit lower="-0.785" upper="0.785" effort="10" velocity="10" />
+    </joint>
+    <link name="left_front_wheel">
+        <inertial>
+            <xacro:wheels_inertial_params z_offset="0"/>
+        </inertial>
+        <visual>
+            <xacro:wheel_geometry prefix="left_front" />
+        </visual>
+        <collision>
+           <xacro:wheel_collision_geometry />
+        </collision>
+    </link>
+    <joint name="left_front_wheel_joint" type="continuous">
+        <origin xyz="0 0 0" rpy="${pi/2} 0 0" />
+        <parent link="left_steering_hinge" />
+        <child link="left_front_wheel" />
+        <axis xyz="0 1 0" />
+        <limit effort="10" velocity="100" />
+    </joint>
+    <link name="right_front_wheel">
+        <inertial>
+           <xacro:wheels_inertial_params z_offset="0"/>
+        </inertial>
+        <visual>
+            <xacro:wheel_geometry prefix="right_front" />
+        </visual>
+        <collision>
+            <xacro:wheel_collision_geometry />
+        </collision>
+    </link>
+    <joint name="right_front_wheel_joint" type="continuous">
+        <origin xyz="0 0 0"  rpy="${pi/2} 0 ${pi}" />
+        <parent link="right_steering_hinge" />
+        <child link="right_front_wheel" />
+        <axis xyz="0 1 0" />
+        <limit effort="10" velocity="100"/>
+    </joint>
+    <xacro:include filename="$(find car_description)/urdf/material.xacro" />
+    <gazebo>
+        <plugin name="gazebo_ros2_control" filename="libgazebo_ros2_control.so">
+            <parameters>$(find car_description)/config/ackermann_control.yaml</parameters>
+            <robot_namespace>/my_ackermann</robot_namespace>
+        </plugin>
+    </gazebo>
+    <!-- <transmission name="left_rear_trans">
+        <type>transmission_interface/SimpleTransmission</type>
+        <joint name="left_rear_wheel_joint">
+          <hardwareInterface>hardware_interface/VelocityJointInterface</hardwareInterface>
+        </joint>
+        <actuator name="left_rear_motor">
+          <hardwareInterface>hardware_interface/VelocityJointInterface</hardwareInterface>
+          <mechanicalReduction>1</mechanicalReduction>
+        </actuator>
+    </transmission>
+    <transmission name="right_rear_trans">
+        <type>transmission_interface/SimpleTransmission</type>
+        <joint name="right_rear_wheel_joint">
+          <hardwareInterface>hardware_interface/VelocityJointInterface</hardwareInterface>
+        </joint>
+        <actuator name="right_rear_motor">
+          <hardwareInterface>hardware_interface/VelocityJointInterface</hardwareInterface>
+          <mechanicalReduction>1</mechanicalReduction>
+        </actuator>
+    </transmission>
+    <transmission name="left_steering_trans">
+        <type>transmission_interface/SimpleTransmission</type>
+        <joint name="left_steering_hinge_joint">
+          <hardwareInterface>hardware_interface/PositionJointInterface</hardwareInterface>
+        </joint>
+        <actuator name="left_steering_motor">
+          <hardwareInterface>hardware_interface/PositionJointInterface</hardwareInterface>
+          <mechanicalReduction>1</mechanicalReduction>
+        </actuator>
+    </transmission>
+    <transmission name="right_steering_trans">
+        <type>transmission_interface/SimpleTransmission</type>
+        <joint name="right_steering_hinge_joint">
+          <hardwareInterface>hardware_interface/PositionJointInterface</hardwareInterface>
+        </joint>
+        <actuator name="right_steering_motor">
+          <hardwareInterface>hardware_interface/PositionJointInterface</hardwareInterface>
+          <mechanicalReduction>1</mechanicalReduction>
+        </actuator>
+    </transmission>  -->
+    <ros2_control name="f1tenth_mock_hw" type="system">
+      <hardware>
+        <plugin>mock_components/GenericSystem</plugin>
+      </hardware>
+        <!-- Hajtott hátsó kerekek -->
+        <joint name="left_rear_wheel_joint">
+            <command_interface name="velocity"/>
+            <state_interface name="position"/>
+            <state_interface name="velocity"/>
+        </joint>
+        <joint name="right_rear_wheel_joint">
+            <command_interface name="velocity"/>
+            <state_interface name="position"/>
+            <state_interface name="velocity"/>
+        </joint>
+        <!-- Kormányzott első csuklók -->
+        <joint name="left_steering_hinge_joint">
+            <command_interface name="position"/>
+            <state_interface name="position"/>
+            <state_interface name="velocity"/>
+        </joint>
+        <joint name="right_steering_hinge_joint">
+            <command_interface name="position"/>
+            <state_interface name="position"/>
+            <state_interface name="velocity"/>
+        </joint>
+        <!-- Passzív első kerekek csak TF-re -->
+        <joint name="left_front_wheel_joint">
+            <state_interface name="position"/>
+            <state_interface name="velocity"/>
+        </joint>
+        <joint name="right_front_wheel_joint">
+            <state_interface name="position"/>
+            <state_interface name="velocity"/>
+        </joint>
+    </ros2_control>
+</robot>

File: install/car_description/share/car_description/urdf/macros.xacro (robot description, xacro)
@@ -1 +1,67 @@
-/home/ezo/f1tenth_ws/build/car_description/urdf/macros.xacro
+<?xml version="1.0"?>
+<robot name="racecar" xmlns:xacro="http://www.ros.org/wiki/xacro">
+<!-- Define the parameters for the car -->
+  <xacro:arg name="wheel_radius" default="0.05" />
+  <xacro:arg name="wheel_separation" default="0.32" />
+  <xacro:arg name="wheelbase" default="0.235" />
+  <xacro:arg name="wheel_width" default="0.045"/>
+  <xacro:arg name="chassis_mass" default="1.0" />
+  <xacro:arg name="wheel_mass" default="0.3" />
+  <xacro:arg name="steering_hinge_mass" default="0.1" />
+  <xacro:property name="wheel_radius" value="$(arg wheel_radius)" />
+  <xacro:property name="wheel_separation" value="$(arg wheel_separation)" />
+  <xacro:property name="wheelbase" value="$(arg wheelbase)" />
+  <xacro:property name="wheel_width" value="$(arg wheel_width)" />
+  <xacro:property name="chassis_mass" value="$(arg chassis_mass)" />
+  <xacro:property name="wheel_mass" value="$(arg wheel_mass)" />
+  <xacro:property name="steering_hinge_mass" value="$(arg steering_hinge_mass)" />
+<!-- chassis geometry-->
+<xacro:macro name="chassis_geometry">
+  <origin xyz="0 0 0" rpy="0 0 0" />
+  <geometry>
+    <mesh filename="package://car_description/meshes/chassis.stl" scale="0.001 0.001 0.001"/>
+  </geometry>
+  <material name="red" />
+</xacro:macro>
+<!-- wheels geometry-->
+<xacro:macro name="wheel_geometry" params="prefix">
+  <origin xyz="0 0 0" rpy="0 0 0" />
+  <geometry>
+    <mesh filename="package://car_description/meshes/wheel.stl" scale="0.001 0.001 0.001"/>
+  </geometry>
+  <material name="black" />
+</xacro:macro>
+<!-- wheels geometry collision-->
+<xacro:macro name="wheel_collision_geometry">
+    <geometry>
+      <mesh filename="package://car_description/meshes/wheel.stl" scale="0.001 0.001 0.001"/>
+    </geometry>
+</xacro:macro>
+<!-- steering hinge geometry -->
+<xacro:macro name="steering_hinge_geometry" params="prefix">
+  <origin xyz="0 0 0" rpy="0 0 0" />
+  <geometry>
+    <mesh filename="package://car_description/meshes/steering_hinge.stl" scale="0.001 0.001 0.001"/>
+  </geometry>
+  <material name="grey" />
+</xacro:macro>
+<!-- inertial parameter macros -->
+<xacro:macro name="chassis_inertial_params">
+  <origin xyz="0 0 0" rpy="0 0 0" />
+  <mass value="${chassis_mass}" />
+  <inertia  ixx="0.1" ixy="0"  ixz="0"
+            iyy="0.1" iyz="0"  izz="0.1" />
+</xacro:macro>
+<xacro:macro name="wheels_inertial_params" params="z_offset">
+  <origin xyz="0 0 ${z_offset}" rpy="0 0 0" />
+  <mass value="${wheel_mass}" />
+  <inertia  ixx="0.1" ixy="0"  ixz="0"
+            iyy="0.1" iyz="0"  izz="0.1" />
+</xacro:macro>
+<xacro:macro name="steering_hinge_inertial_params" params="z_offset">
+  <origin xyz="0 0 ${z_offset}" rpy="0 0 0" />
+  <mass value="${steering_hinge_mass}" />
+  <inertia  ixx="0.1" ixy="0"  ixz="0"
+            iyy="0.1" iyz="0"  izz="0.1" />
+</xacro:macro>
+</robot>

File: install/car_description/share/car_description/urdf/material.xacro (robot description, xacro)
@@ -1 +1,27 @@
-/home/ezo/f1tenth_ws/build/car_description/urdf/material.xacro
+<?xml version="1.0"?>
+<robot name="racecar" xmlns:xacro="http://www.ros.org/wiki/xacro">
+<material name="black">
+  <color rgba="0.0 0.0 0.0 1.0"/>
+</material>
+<material name="blue">
+  <color rgba="0.0 0.0 0.8 1.0"/>
+</material>
+<material name="green">
+  <color rgba="0.0 0.8 0.0 1.0"/>
+</material>
+<material name="grey">
+  <color rgba="0.2 0.2 0.2 1.0"/>
+</material>
+<material name="orange">
+  <color rgba="${255/255} ${108/255} ${10/255} 1.0"/>
+</material>
+<material name="brown">
+  <color rgba="${222/255} ${207/255} ${195/255} 1.0"/>
+</material>
+<material name="red">
+  <color rgba="0.8 0.0 0.0 1.0"/>
+</material>
+<material name="white">
+  <color rgba="1.0 1.0 1.0 1.0"/>
+</material>
+</robot>

File: src/car_description/urdf/base_link.xacro (robot description, xacro)
@@ -136,38 +136,79 @@
         </plugin>
     </gazebo>
+    <!-- <transmission name="left_rear_trans">
+        <type>transmission_interface/SimpleTransmission</type>
+        <joint name="left_rear_wheel_joint">
+          <hardwareInterface>hardware_interface/VelocityJointInterface</hardwareInterface>
+        </joint>
+        <actuator name="left_rear_motor">
+          <hardwareInterface>hardware_interface/VelocityJointInterface</hardwareInterface>
+          <mechanicalReduction>1</mechanicalReduction>
+        </actuator>
+    </transmission>
+    <transmission name="right_rear_trans">
+        <type>transmission_interface/SimpleTransmission</type>
+        <joint name="right_rear_wheel_joint">
+          <hardwareInterface>hardware_interface/VelocityJointInterface</hardwareInterface>
+        </joint>
+        <actuator name="right_rear_motor">
+          <hardwareInterface>hardware_interface/VelocityJointInterface</hardwareInterface>
+          <mechanicalReduction>1</mechanicalReduction>
+        </actuator>
+    </transmission>
+    <transmission name="left_steering_trans">
+        <type>transmission_interface/SimpleTransmission</type>
+        <joint name="left_steering_hinge_joint">
+          <hardwareInterface>hardware_interface/PositionJointInterface</hardwareInterface>
+        </joint>
+        <actuator name="left_steering_motor">
+          <hardwareInterface>hardware_interface/PositionJointInterface</hardwareInterface>
+          <mechanicalReduction>1</mechanicalReduction>
+        </actuator>
+    </transmission>
+    <transmission name="right_steering_trans">
+        <type>transmission_interface/SimpleTransmission</type>
+        <joint name="right_steering_hinge_joint">
+          <hardwareInterface>hardware_interface/PositionJointInterface</hardwareInterface>
+        </joint>
+        <actuator name="right_steering_motor">
+          <hardwareInterface>hardware_interface/PositionJointInterface</hardwareInterface>
+          <mechanicalReduction>1</mechanicalReduction>
+        </actuator>
+    </transmission>  -->
     <ros2_control name="f1tenth_mock_hw" type="system">
       <hardware>
         <plugin>mock_components/GenericSystem</plugin>
       </hardware>
-      <joint name="right_rear_wheel_joint">
-        <command_interface name="velocity"/>
-        <state_interface name="position"/>
-        <state_interface name="velocity"/>
-      </joint>
-      <joint name="left_rear_wheel_joint">
-        <command_interface name="velocity"/>
-        <state_interface name="velocity"/>
-        <state_interface name="position"/>
-      </joint>
-      <joint name="right_steering_hinge_joint">
-        <command_interface name="position"/>
-        <state_interface name="velocity"/>
-        <state_interface name="position"/>
-      </joint>
-      <joint name="left_steering_hinge_joint">
-        <command_interface name="position"/>
-        <state_interface name="velocity"/>
-        <state_interface name="position"/>
-      </joint>
-      <joint name="left_front_wheel_joint">
+        <!-- Hajtott hátsó kerekek -->
+        <joint name="left_rear_wheel_joint">
             <command_interface name="velocity"/>
             <state_interface name="position"/>
             <state_interface name="velocity"/>
-      </joint>
-      <joint name="right_front_wheel_joint">
+        </joint>
+        <joint name="right_rear_wheel_joint">
             <command_interface name="velocity"/>
             <state_interface name="position"/>
             <state_interface name="velocity"/>
-      </joint>
+        </joint>
+        <!-- Kormányzott első csuklók -->
+        <joint name="left_steering_hinge_joint">
+            <command_interface name="position"/>
+            <state_interface name="position"/>
+            <state_interface name="velocity"/>
+        </joint>
+        <joint name="right_steering_hinge_joint">
+            <command_interface name="position"/>
+            <state_interface name="position"/>
+            <state_interface name="velocity"/>
+        </joint>
+        <!-- Passzív első kerekek csak TF-re -->
+        <joint name="left_front_wheel_joint">
+            <state_interface name="position"/>
+            <state_interface name="velocity"/>
+        </joint>
+        <joint name="right_front_wheel_joint">
+            <state_interface name="position"/>
+            <state_interface name="velocity"/>
+        </joint>
     </ros2_control>
 </robot>
